Commit message: [20240805]xacro学习

File: src/urdf01_rviz/urdf/urdf/demo05_test.urdf (robot description, URDF)
Before this commit: robot mycar, 4 links, 3 joints
Links:
- removed link left_whell
- removed link right_whell
- added link back_wheel; visual sphere radius=0.0075
- added link front_wheel; visual sphere radius=0.0075
- added link left_wheel; visual cylinder length=0.015 radius=0.0325
- added link right_wheel; visual cylinder length=0.015 radius=0.0325
Joints:
- added joint back2link: type continuous, parent base_link, child back_wheel, origin xyz=-0.08 0 -0.0475 rpy=0 0 0, axis 0 1 0
- added joint front2link: type continuous, parent base_link, child front_wheel, origin xyz=0.08 0 -0.0475 rpy=0 0 0, axis 0 1 0
- joint left2link: child left_whell -> left_wheel
- joint right2link: child right_whell -> right_wheel
