Commit message: [20240806]gazebo集成 1.报错Shutdown request received. 2.报错Reason given for shutdown: [[/gazebo_gui] Reason: new node registered with same name] 3.报错[ WARN] [1722933405.733183230, 257.802000000]: DiffDrive(ns = //): missing <odometrySource> default is 1

File: src/urdf02_gazebo/urdf/car.urdf.xacro (robot description, xacro)
@@ -4,3 +4,4 @@
     <xacro:include filename="demo06_car_camera.urdf.xacro"/>
     <xacro:include filename="demo07_car_laser.urdf.xacro"/>
+    <xacro:include filename="gazebo/move.xacro"/>
 </robot>

File: src/urdf02_gazebo/urdf/demo05_car_base.urdf.xacro (robot description, xacro)
@@ -10,5 +10,5 @@
     <xacro:property name="base_radius" value="0.1"/>
     <xacro:property name="base_length" value="0.08"/>
-    <xacro:property name="base_mass" value="2"/>
+    <xacro:property name="base_mass" value="1"/>
     <xacro:property name="lidi" value="0.015"/>
     <xacro:property name="base_joint_z" value="${base_length / 2 +lidi}"/>
@@ -41,5 +41,5 @@
     <xacro:property name="wheel_radius" value="0.0325"/>
     <xacro:property name="wheel_length" value="0.015"/>
-    <xacro:property name="wheel_mass" value="0.005"/>
+    <xacro:property name="wheel_mass" value="0.05"/>
     <xacro:property name="PI" value="3.1415927"/>
     <xacro:property name="wheel_joint_z" value="${(base_length / 2 + lidi - wheel_radius) * -1}"/>

File: src/urdf02_gazebo/urdf/demo06_car_camera.urdf.xacro (robot description, xacro)
@@ -3,4 +3,5 @@
     <xacro:property name="camera_width" value="0.05"/>
     <xacro:property name="camera_height" value="0.05"/>
+    <xacro:property name="camera_mass" value="0.01"/>
     <xacro:property name="joint_camera_x" value="0.08"/>
     <xacro:property name="joint_camera_y" value="0"/>
@@ -15,5 +16,14 @@
             </material>
         </visual>
+        <collision>
+            <geometry>
+                <box size="${camera_lenght} ${camera_width} ${camera_height}"/>
+            </geometry>
+        </collision>
+        <xacro:Box_inertial_matrix m="${camera_mass}" l="${camera_lenght}" w="${camera_width}" h="${camera_height}"/>
     </link>
+    <gazebo reference="camera">
+        <material>Gazebo/Blue</material>
+    </gazebo>
     <joint name="camera2base" type="fixed">
         <parent link="base_link"/>

File: src/urdf02_gazebo/urdf/demo07_car_laser.urdf.xacro (robot description, xacro)
@@ -2,6 +2,8 @@
     <xacro:property name="support_radius" value="0.01"/>
     <xacro:property name="support_length" value="0.15"/>
+    <xacro:property name="support_mass" value="0.1"/>
     <xacro:property name="laser_radius" value="0.03"/>
     <xacro:property name="laser_length" value="0.05"/>
+    <xacro:property name="laser_mass" value="0.15"/>
     <xacro:property name="joint_support_x" value="0"/>
     <xacro:property name="joint_support_y" value="0"/>
@@ -19,5 +21,14 @@
             </material>
         </visual>
+        <collision>
+            <geometry>
+                <cylinder radius="${support_radius}" length="${support_length}"/>
+            </geometry>
+        </collision>
+        <xacro:cylinder_inertial_matrix m="${support_mass}" r="${support_radius}" h="${support_length}"/>
     </link>
+    <gazebo reference="support">
+        <material>Gazebo/Gray</material>
+    </gazebo>
     <joint name="support2base" type="fixed">
         <origin xyz="${joint_support_x} ${joint_support_y} ${joint_support_z}" rpy="0 0 0"/>
@@ -34,5 +45,14 @@
             </material>
         </visual>
+        <collision>
+            <geometry>
+                <cylinder radius="${laser_radius}" length="${laser_length}"/>
+            </geometry>
+        </collision>
+        <xacro:cylinder_inertial_matrix m="${laser_mass}" r="${laser_radius}" h="${laser_length}"/>
     </link>
+    <gazebo reference="laser">
+        <material>Gazebo/Blue</material>
+    </gazebo>
     <joint name="laser2support" type="fixed">
         <origin xyz="${joint_laser_x} ${joint_laser_y} ${joint_laser_z}" rpy="0 0 0"/>
